File: pcb/astrasat1/astrasat1.kicad_sch (KiCad schematic)
At the start: 16 parts, among them M1 Motor_Servo, U2 MPU-6050, U7 DS1302+, U9 Pico, Y1 Crystal

Commit message: save and export minor revision
Parts:
- added SW1: SW_SPDT, symbol Switch:SW_SPDT
Connections:
- net at BT1.1 (+), BT2.1 (+), BT3.1 (+): now also SW1.2 (B); no longer M1.2 (+), U1. (OUT-)
- new net: M1.2 (+), SW1.1 (A), U1. (OUT-)
Other:
- moved on the sheet: BT1, BT2, BT3, M1
