File: pcb/astrasat1/astrasat1.kicad_pcb (KiCad board)
At the start: 2 copper layers, 120 x 120 mm, 22 parts, among them SW1 SW_SPDT, U3 DS1302+, U5 Pico, Y1 Crystal

Commit message: update
Parts:
- added G***: LOGO, CansatFootprints:POLITOLogo, B.Cu at (109.2, 94.0)
- added G***: LOGO, CansatFootprints:ASTRALogo, B.Cu at (205.7, 94.0)
- added REF**: Symbol_GNU-Logo_SilkscreenTop, Symbol:Symbol_GNU-Logo_SilkscreenTop, F.Cu at (111.8, 70.2)
Routing:
- net VSYS: track 254.5 -> 320.6 mm, vias 0 -> 2
- net /GPIO6: track 0.00 -> 47.0 mm, vias 0 -> 2
- net GND2: track 55.3 -> 54.6 mm
Other:
- board text added: "ASTRASAT PICO V1"
- board text added: "PCB designed by Tan S. Akıncı"

Commit message: edit pcb and generate gerber files
Parts:
- added G***: LOGO, CansatFootprints:ASTRAIcon, F.Cu at (152.0, 150.7)
- REF**: moved to B.Cu
- moved REF** 82.7 mm to (151.8, 142.6)
