File: pcb/astrasat1/astrasat1.kicad_pcb (KiCad board)
At the start: 2 copper layers, 120 x 120 mm, 26 parts, among them SW1 SW_SPDT, U3 DS1302+, U5 Pico, Y1 Crystal

Commit message: update
Parts:
- moved REF** 12.7 mm to (151.8, 129.9)
Changed lines of the file:
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@@
   )
   (footprint "Symbol:Symbol_GNU-Logo_SilkscreenTop" (layer "B.Cu")
-    (at 151.78481 142.56893 180)
+    (at 151.78481 129.86893 180)
     (descr "GNU-Logo, GNU-Head, GNU-Kopf, Silkscreen,")
     (tags "GNU-Logo, GNU-Head, GNU-Kopf, Silkscreen,")
@@
   (gr_circle (center 151.815 94.36) (end 211.815 94.36)
     (stroke (width 0.1) (type default)) (fill none) (layer "Edge.Cuts"))
-  (gr_text "PCB designed by \nTan S. Akıncı" (at 152.035 151.765) (layer "B.SilkS")
+  (gr_text "PCB designed by \nTan S. Akıncı" (at 152.035 139.065) (layer "B.SilkS")
     (effects (font (size 0.8 0.8) (thickness 0.1)) (justify bottom))
   )
