File: astrasat_pcb/astrasat1.kicad_pcb (KiCad board)
At the start: 2 copper layers, 120 x 120 mm, 28 parts, among them SW1 SW_SPDT, U3 DS1302+, U5 Pico, Y1 Crystal

Commit message: reduce pcb size
Parts:
- moved MainBT1 4.53 mm to (181.6, 142.2)
- moved Y1 0.93 mm to (180.3, 45.7)
- moved U6 0.90 mm to (112.4, 87.3)
- moved REF** 0.64 mm to (109.9, 57.7)
- moved REF** 0.64 mm to (109.9, 130.8)
- moved SW1 0.48 mm to (178.5, 139.7)
- moved U3 0.36 mm to (188.0, 50.5)
- moved REF** 0.32 mm to (193.7, 130.8)
- moved REF** 0.32 mm to (193.7, 57.7)
- moved G*** 0.20 mm to (152.0, 150.5)
Routing:
- net Net-(MainBT1-+): track 8.05 -> 0.00 mm
- net Net-(D2-A): track 4.59 -> 0.04 mm
- net GND2: track 54.6 -> 55.9 mm
- net Net-(U3-X1): track 7.17 -> 6.12 mm
- net Net-(U3-X2): track 6.90 -> 5.85 mm
- net /GPIO9: track 78.5 -> 77.6 mm
- net /GPIO11: track 70.5 -> 69.6 mm
- net /GPIO10: track 51.1 -> 50.2 mm
- net /GPIO8: track 60.0 -> 59.1 mm
Other:
- board size 120 x 120 mm -> 118 x 118 mm

Commit message: update
Parts:
- added SmallM2: Motor_Servo, Connector_PinHeader_2.54mm:PinHeader_1x03_P2.54mm_Vertical, F.Cu at (207.0, 87.0)
- added SmallM3: Motor_Servo, Connector_PinHeader_2.54mm:PinHeader_1x03_P2.54mm_Vertical, F.Cu at (207.0, 93.3)
- moved G*** 75.4 mm to (152.4, 40.6), turned to 180 degrees
Connections:
- U5 pad 6: unconnected-(U5-GPIO4-Pad6) -> /GPIO4
- U5 pad 7: unconnected-(U5-GPIO5-Pad7) -> /GPIO5
Routing:
- net /GPIO4: track 0.00 -> 73.9 mm
- net /GPIO5: track 0.00 -> 69.2 mm, vias 0 -> 2
- net VSYS: track 320.6 -> 329.7 mm

Commit message: Update PCB
Parts:
- added J1: CAM1, Connector_PinHeader_2.54mm:PinHeader_1x03_P2.54mm_Vertical, F.Cu at (117.9, 124.5)
- added J2: CAM2, Connector_PinHeader_2.54mm:PinHeader_1x03_P2.54mm_Vertical, F.Cu at (122.6, 124.5)
- moved SW1 0.97 mm to (177.5, 139.8)
Connections:
- SmallM2 pad 1: /GPIO5 -> /GPIO1
- SmallM3 pad 1: /GPIO4 -> /GPIO0
- U4 pad 2: /GPIO0 -> /GPIO4
- U4 pad 3: /GPIO1 -> /GPIO5
- U5 pad 24: unconnected-(U5-GPIO18-Pad24) -> /GPIO18
- U5 pad 25: unconnected-(U5-GPIO19-Pad25) -> /GPIO19
Routing:
- net /GPIO18: track 0.00 -> 53.1 mm, vias 0 -> 1
- net /GPIO19: track 0.00 -> 34.2 mm, vias 0 -> 1
- net /GPIO0: track 99.0 -> 82.2 mm, vias 2 -> 1
- net VSYS: track 329.7 -> 342.4 mm
- net /GPIO5: track 69.2 -> 81.3 mm
- net /GPIO1: track 94.0 -> 82.0 mm, vias 2 -> 3
- net /GPIO4: track 73.9 -> 85.6 mm, vias 0 -> 2
- net Net-(D2-A): track 0.04 -> 5.62 mm
- net Net-(MainBT1-+): track 0.00 -> 4.15 mm
