File: astrasat_pcb/astrasat1.kicad_sch (KiCad schematic)
At the start: 17 parts, among them SW1 SW_SPDT, U3 DS1302+, U5 Pico, Y1 Crystal

Commit message: update
Parts:
- added SmallM2, SmallM3: Motor_Servo, Connector_PinHeader_2.54mm:PinHeader_1x03_P2.54mm_Vertical, symbol Motor:Motor_Servo
Connections:
- net GND1: now also SmallM2.3 (-), SmallM3.3 (-)
- net VSYS: now also SmallM2.2 (+), SmallM3.2 (+)
- net GPIO4: now reaches U5.6 (GPIO4)
- net GPIO4: now also SmallM3.1 (PWM)
- net GPIO5: now reaches U5.7 (GPIO5)
- net GPIO5: now also SmallM2.1 (PWM)
- no-connect marks 43 -> 41
Changed lines of the file:
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@@
   (title_block
     (title "ASTRASAT PCB")
-    (date "2023-11-23")
-    (rev "v1.02.5")
+    (date "2023-11-29")
+    (rev "v1.02.6")
     (comment 3 "                                                                    License: CC BY-SA 4.0")
     (comment 4 "                                                                    Author: Tan Siret Akıncı")
@@
   (no_connect (at 109.22 116.205))
   (no_connect (at 120.65 73.66))
-  (no_connect (at 127 156.845))
   (no_connect (at 167.005 153.035))
-  (no_connect (at 127 154.305))
   (no_connect (at 95.25 76.2))
   (no_connect (at 167.005 155.575))
@@
     (stroke (width 0) (type default))
   )
+  (wire (pts (xy 233.68 71.12) (xy 239.395 71.12))
+    (stroke (width 0) (type default))
+  )
   (wire (pts (xy 91.44 133.985) (xy 89.535 133.985))
     (stroke (width 0) (type default))
@@
     (stroke (width 0) (type default))
   )
+  (wire (pts (xy 233.68 60.325) (xy 239.395 60.325))
+    (stroke (width 0) (type default))
+  )
   (wire (pts (xy 127 169.545) (xy 129.54 169.545))
     (stroke (width 0) (type default))
@@
     (stroke (width 0) (type default))
   )
+  (wire (pts (xy 127 156.845) (xy 129.54 156.845))
+    (stroke (width 0) (type default))
+  )
   (wire (pts (xy 35.56 61.595) (xy 26.035 61.595))
     (stroke (width 0) (type default))
@@
     (stroke (width 0) (type default))
   )
+  (wire (pts (xy 236.855 73.66) (xy 239.395 73.66))
+    (stroke (width 0) (type default))
+  )
   (wire (pts (xy 228.6 94.615) (xy 228.6 109.855))
     (stroke (width 0) (type default))
@@
     (stroke (width 0) (type default))
   )
+  (wire (pts (xy 237.49 68.58) (xy 239.395 68.58))
+    (stroke (width 0) (type default))
+  )
   (wire (pts (xy 91.44 121.285) (xy 89.535 121.285))
     (stroke (width 0) (type default))
@@
     (stroke (width 0) (type default))
   )
+  (wire (pts (xy 127 154.305) (xy 129.54 154.305))
+    (stroke (width 0) (type default))
+  )
   (wire (pts (xy 128.27 136.525) (xy 127 136.525))
     (stroke (width 0) (type default))
@@
     (stroke (width 0) (type default))
   )
+  (wire (pts (xy 237.49 57.785) (xy 239.395 57.785))
+    (stroke (width 0) (type default))
+  )
   (wire (pts (xy 193.04 114.3) (xy 203.835 114.3))
     (stroke (width 0) (type default))
@@
     (stroke (width 0) (type default))
   )
+  (wire (pts (xy 236.855 62.865) (xy 239.395 62.865))
+    (stroke (width 0) (type default))
+  )
   (wire (pts (xy 48.895 24.13) (xy 48.895 27.94))
     (stroke (width 0) (type default))
@@
     (effects (font (size 1.27 1.27)) (justify right bottom))
   )
+  (label "GPIO5" (at 129.54 154.305 0) (fields_autoplaced)
+    (effects (font (size 1.27 1.27)) (justify left bottom))
+  )
   (label "GPIO21" (at 63.5 43.18 0) (fields_autoplaced)
     (effects (font (size 1.27 1.27)) (justify left bottom))
@@
     (effects (font (size 1.27 1.27)) (justify left bottom))
   )
+  (label "GPIO4" (at 237.49 57.785 180) (fields_autoplaced)
+    (effects (font (size 1.27 1.27)) (justify right bottom))
+  )
   (label "GPIO7" (at 129.54 146.685 0) (fields_autoplaced)
     (effects (font (size 1.27 1.27)) (justify left bottom))
@@
   )
   (label "GPIO17" (at 45.72 142.24 0) (fields_autoplaced)
+    (effects (font (size 1.27 1.27)) (justify left bottom))
+  )
+  (label "GPIO5" (at 237.49 68.58 180) (fields_autoplaced)
+    (effects (font (size 1.27 1.27)) (justify right bottom))
+  )
+  (label "GPIO4" (at 129.54 156.845 0) (fields_autoplaced)
     (effects (font (size 1.27 1.27)) (justify left bottom))
   )
@@
     )
   )
+  (global_label "VSYS" (shape input) (at 233.68 60.325 180) (fields_autoplaced)
+    (effects (font (size 1.27 1.27)) (justify right))
+    (property "Intersheetrefs" "${INTERSHEET_REFS}" (at 226.0986 60.325 0)
+      (effects (font (size 1.27 1.27)) (justify right) hide)
+    )
+  )
   (global_label "VSYS" (shape input) (at 53.34 115.57 0) (fields_autoplaced)
     (effects (font (size 1.27 1.27)) (justify left))
@@
     )
   )
+  (global_label "VSYS" (shape input) (at 233.68 71.12 180) (fields_autoplaced)
+    (effects (font (size 1.27 1.27)) (justify right))
+    (property "Intersheetrefs" "${INTERSHEET_REFS}" (at 226.0986 71.12 0)
+      (effects (font (size 1.27 1.27)) (justify right) hide)
+    )
+  )
   (symbol (lib_id "power:GND1") (at 193.04 114.3 270) (unit 1)
     (in_bom yes) (on_board yes) (dnp no) (fields_autoplaced)
@@
         (path "/9e2da17e-9926-4640-a42c-f97fd7426e13"
           (reference "#PWR04") (unit 1)
+        )
+      )
+    )
+  )
+  (symbol (lib_id "Motor:Motor_Servo") (at 247.015 71.12 0) (unit 1)
+    (in_bom yes) (on_board yes) (dnp no) (fields_autoplaced)
+    (property "Reference" "SmallM2" (at 256.54 69.4166 0)
+      (effects (font (size 1.27 1.27)) (justify left))
+    )
+    (property "Value" "Motor_Servo" (at 256.54 71.9566 0)
+      (effects (font (size 1.27 1.27)) (justify left))
+    )
+    (property "Footprint" "Connector_PinHeader_2.54mm:PinHeader_1x03_P2.54mm_Vertical" (at 247.015 75.946 0)
+      (effects (font (size 1.27 1.27)) hide)
+    )
+    (property "Datasheet" "http://forums.parallax.com/uploads/attachments/46831/74481.png" (at 247.015 75.946 0)
+      (effects (font (size 1.27 1.27)) hide)
+    )
+    (pin "2")
+    (pin "3")
+    (pin "1")
+    (instances
+      (project "astrasat1"
+        (path "/9e2da17e-9926-4640-a42c-f97fd7426e13"
+          (reference "SmallM2") (unit 1)
         )
       )
@@
     )
   )
+  (symbol (lib_id "power:GND1") (at 236.855 62.865 270) (unit 1)
+    (in_bom yes) (on_board yes) (dnp no) (fields_autoplaced)
+    (property "Reference" "#PWR021" (at 230.505 62.865 0)
+      (effects (font (size 1.27 1.27)) hide)
+    )
+    (property "Value" "GND1" (at 233.045 62.865 90)
+      (effects (font (size 1.27 1.27)) (justify right))
+    )
+    (property "Footprint" "" (at 236.855 62.865 0)
+      (effects (font (size 1.27 1.27)) hide)
+    )
+    (property "Datasheet" "" (at 236.855 62.865 0)
+      (effects (font (size 1.27 1.27)) hide)
+    )
+    (pin "1")
+    (instances
+      (project "astrasat1"
+        (path "/9e2da17e-9926-4640-a42c-f97fd7426e13"
+          (reference "#PWR021") (unit 1)
+        )
+      )
+    )
+  )
   (symbol (lib_id "Device:Battery_Cell") (at 261.62 140.335 90) (unit 1)
     (in_bom yes) (on_board yes) (dnp no) (fields_autoplaced)
@@
     )
   )
+  (symbol (lib_id "Motor:Motor_Servo") (at 247.015 60.325 0) (unit 1)
+    (in_bom yes) (on_board yes) (dnp no) (fields_autoplaced)
+    (property "Reference" "SmallM3" (at 256.54 58.6216 0)
+      (effects (font (size 1.27 1.27)) (justify left))
+    )
+    (property "Value" "Motor_Servo" (at 256.54 61.1616 0)
+      (effects (font (size 1.27 1.27)) (justify left))
+    )
+    (property "Footprint" "Connector_PinHeader_2.54mm:PinHeader_1x03_P2.54mm_Vertical" (at 247.015 65.151 0)
+      (effects (font (size 1.27 1.27)) hide)
+    )
+    (property "Datasheet" "http://forums.parallax.com/uploads/attachments/46831/74481.png" (at 247.015 65.151 0)
+      (effects (font (size 1.27 1.27)) hide)
+    )
+    (pin "2")
+    (pin "3")
+    (pin "1")
+    (instances
+      (project "astrasat1"
+        (path "/9e2da17e-9926-4640-a42c-f97fd7426e13"
+          (reference "SmallM3") (unit 1)
+        )
+      )
+    )
+  )
   (symbol (lib_id "power:GND1") (at 136.525 92.075 0) (unit 1)
     (in_bom yes) (on_board yes) (dnp no) (fields_autoplaced)
@@
         )
       )
+    )
+  )
+  (symbol (lib_id "power:GND1") (at 236.855 73.66 270) (unit 1)
+    (in_bom yes) (on_board yes) (dnp no) (fields_autoplaced)
+    (property "Reference" "#PWR020" (at 230.505 73.66 0)
+      (effects (font (size 1.27 1.27)) hide)
+    )
+    (property "Value" "GND1" (at 233.045 73.66 90)
+      (effects (font (size 1.27 1.27)) (justify right))
+    )
+    (property "Footprint" "" (at 236.855 73.66 0)
+      (effects (font (size 1.27 1.27)) hide)
+    )
+    (property "Datasheet" "" (at 236.855 73.66 0)
+      (effects (font (size 1.27 1.27)) hide)
+    )
+    (pin "1")
+    (instances
+      (project "astrasat1"
+        (path "/9e2da17e-9926-4640-a42c-f97fd7426e13"
+          (reference "#PWR020") (unit 1)
+        )
+      )

Commit message: Update PCB
Parts:
- added J1: CAM1, Connector_PinHeader_2.54mm:PinHeader_1x03_P2.54mm_Vertical, symbol Connector:Conn_01x03_Pin
- added J2: CAM2, Connector_PinHeader_2.54mm:PinHeader_1x03_P2.54mm_Vertical, symbol Connector:Conn_01x03_Pin
Connections:
- net GND1: now also J1.3 (Pin_3), J2.3 (Pin_3)
- net GPIO0: now also SmallM3.1 (PWM); no longer U4.2 (DOUT)
- net GPIO1: now also SmallM2.1 (PWM); no longer U4.3 (DIN/~{CON})
- net GPIO4: now also U4.2 (DOUT); no longer SmallM3.1 (PWM)
- net GPIO5: now also U4.3 (DIN/~{CON}); no longer SmallM2.1 (PWM)
- net VSYS: now also J1.1 (Pin_1), J2.1 (Pin_1)
- net GPIO18: now reaches U5.24 (GPIO18)
- net GPIO18: now also J1.2 (Pin_2)
- net GPIO19: now reaches U5.25 (GPIO19)
- net GPIO19: now also J2.2 (Pin_2)
- no-connect marks 41 -> 39
Changed lines of the file:
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@@
   (title_block
     (title "ASTRASAT PCB")
-    (date "2023-11-29")
-    (rev "v1.02.6")
+    (date "2023-12-14")
+    (rev "v1.02.7")
     (comment 3 "                                                                    License: CC BY-SA 4.0")
     (comment 4 "                                                                    Author: Tan Siret Akıncı")
@@
   (no_connect (at 91.44 149.225))
   (no_connect (at 95.25 73.66))
-  (no_connect (at 91.44 131.445))
   (no_connect (at 149.225 83.82))
   (no_connect (at 111.76 116.205))
@@
   (no_connect (at 120.65 78.74))
   (no_connect (at 167.005 140.335))
-  (no_connect (at 91.44 128.905))
   (no_connect (at 120.65 55.88))
   (no_connect (at 199.39 148.59))
@@
     (stroke (width 0) (type default))
   )
+  (wire (pts (xy 43.815 180.34) (xy 46.99 180.34))
+    (stroke (width 0) (type default))
+  )
   (wire (pts (xy 61.595 30.48) (xy 71.755 30.48))
     (stroke (width 0) (type default))
   )
+  (wire (pts (xy 43.815 162.56) (xy 46.355 162.56))
+    (stroke (width 0) (type default))
+  )
   (wire (pts (xy 91.44 136.525) (xy 89.535 136.525))
     (stroke (width 0) (type default))
@@
     (stroke (width 0) (type default))
   )
+  (wire (pts (xy 89.535 128.905) (xy 91.44 128.905))
+    (stroke (width 0) (type default))
+  )
   (wire (pts (xy 225.425 114.3) (xy 224.155 114.3))
     (stroke (width 0) (type default))
@@
     (stroke (width 0) (type default))
   )
+  (wire (pts (xy 50.8 177.8) (xy 43.815 177.8))
+    (stroke (width 0) (type default))
+  )
   (wire (pts (xy 129.54 161.925) (xy 127 161.925))
     (stroke (width 0) (type default))
@@
     (stroke (width 0) (type default))
   )
+  (wire (pts (xy 43.815 173.355) (xy 43.815 175.26))
+    (stroke (width 0) (type default))
+  )
   (wire (pts (xy 127 154.305) (xy 129.54 154.305))
     (stroke (width 0) (type default))
@@
     (stroke (width 0) (type default))
   )
+  (wire (pts (xy 89.535 131.445) (xy 91.44 131.445))
+    (stroke (width 0) (type default))
+  )
   (wire (pts (xy 45.72 50.165) (xy 48.895 50.165))
     (stroke (width 0) (type default))
@@
     (stroke (width 0) (type default))
   )
+  (wire (pts (xy 50.165 160.02) (xy 43.815 160.02))
+    (stroke (width 0) (type default))
+  )
+  (wire (pts (xy 43.815 155.575) (xy 43.815 157.48))
+    (stroke (width 0) (type default))
+  )
   (wire (pts (xy 237.49 80.01) (xy 239.395 80.01))
     (stroke (width 0) (type default))
@@
     (effects (font (size 1.27 1.27)) (justify right bottom))
   )
-  (label "GPIO0" (at 93.345 58.42 180) (fields_autoplaced)
+  (label "GPIO4" (at 93.345 58.42 180) (fields_autoplaced)
     (effects (font (size 1.27 1.27)) (justify right bottom))
   )
@@
     (effects (font (size 1.27 1.27)) (justify right bottom))
   )
+  (label "GPIO18" (at 89.535 128.905 180) (fields_autoplaced)
+    (effects (font (size 1.27 1.27)) (justify right bottom))
+  )
   (label "GPIO21" (at 89.535 136.525 180) (fields_autoplaced)
     (effects (font (size 1.27 1.27)) (justify right bottom))
@@
     (effects (font (size 1.27 1.27)) (justify left bottom))
   )
-  (label "GPIO1" (at 93.345 60.96 180) (fields_autoplaced)
+  (label "GPIO5" (at 93.345 60.96 180) (fields_autoplaced)
     (effects (font (size 1.27 1.27)) (justify right bottom))
   )
@@
     (effects (font (size 1.27 1.27)) (justify left bottom))
   )
+  (label "GPIO18" (at 50.165 160.02 0) (fields_autoplaced)
+    (effects (font (size 1.27 1.27)) (justify left bottom))
+  )
   (label "GPIO12" (at 128.27 131.445 0) (fields_autoplaced)
     (effects (font (size 1.27 1.27)) (justify left bottom))
@@
     (effects (font (size 1.27 1.27)) (justify right bottom))
   )
+  (label "GPIO19" (at 89.535 131.445 180) (fields_autoplaced)
+    (effects (font (size 1.27 1.27)) (justify right bottom))
+  )
   (label "GPIO17" (at 89.535 123.825 180) (fields_autoplaced)
     (effects (font (size 1.27 1.27)) (justify right bottom))
@@
     (effects (font (size 1.27 1.27)) (justify left bottom))
   )
-  (label "GPIO4" (at 237.49 57.785 180) (fields_autoplaced)
+  (label "GPIO0" (at 237.49 57.785 180) (fields_autoplaced)
     (effects (font (size 1.27 1.27)) (justify right bottom))
   )
@@
     (effects (font (size 1.27 1.27)) (justify left bottom))
   )
+  (label "GPIO19" (at 50.8 177.8 0) (fields_autoplaced)
+    (effects (font (size 1.27 1.27)) (justify left bottom))
+  )
   (label "GPIO7" (at 237.49 80.01 180) (fields_autoplaced)
     (effects (font (size 1.27 1.27)) (justify right bottom))
@@
     (effects (font (size 1.27 1.27)) (justify left bottom))
   )
-  (label "GPIO5" (at 237.49 68.58 180) (fields_autoplaced)
+  (label "GPIO1" (at 237.49 68.58 180) (fields_autoplaced)
     (effects (font (size 1.27 1.27)) (justify right bottom))
   )
@@
     )
   )
+  (global_label "VSYS" (shape input) (at 43.815 173.355 90) (fields_autoplaced)
+    (effects (font (size 1.27 1.27)) (justify left))
+    (property "Intersheetrefs" "${INTERSHEET_REFS}" (at 43.815 165.7736 90)
+      (effects (font (size 1.27 1.27)) (justify left) hide)
+    )
+  )
   (global_label "VSYS" (shape input) (at 55.245 137.16 0) (fields_autoplaced)
     (effects (font (size 1.27 1.27)) (justify left))
@@
     )
   )
+  (global_label "VSYS" (shape input) (at 43.815 155.575 90) (fields_autoplaced)
+    (effects (font (size 1.27 1.27)) (justify left))
+    (property "Intersheetrefs" "${INTERSHEET_REFS}" (at 43.815 147.9936 90)
+      (effects (font (size 1.27 1.27)) (justify left) hide)
+    )
+  )
   (global_label "3V3" (shape input) (at 127 86.995 180) (fields_autoplaced)
     (effects (font (size 1.27 1.27)) (justify right))
@@
     )
   )
+  (symbol (lib_id "power:GND1") (at 46.99 180.34 90) (unit 1)
+    (in_bom yes) (on_board yes) (dnp no)
+    (property "Reference" "#PWR022" (at 53.34 180.34 0)
+      (effects (font (size 1.27 1.27)) hide)
+    )
+    (property "Value" "GND1" (at 50.8 180.34 90)
+      (effects (font (size 1.27 1.27)) (justify right))
+    )
+    (property "Footprint" "" (at 46.99 180.34 0)
+      (effects (font (size 1.27 1.27)) hide)
+    )
+    (property "Datasheet" "" (at 46.99 180.34 0)
+      (effects (font (size 1.27 1.27)) hide)
+    )
+    (pin "1")
+    (instances
+      (project "astrasat1"
+        (path "/9e2da17e-9926-4640-a42c-f97fd7426e13"
+          (reference "#PWR022") (unit 1)
+        )
+      )
+    )
+  )
   (symbol (lib_id "Motor:Motor_Servo") (at 247.015 71.12 0) (unit 1)
     (in_bom yes) (on_board yes) (dnp no) (fields_autoplaced)
@@
         (path "/9e2da17e-9926-4640-a42c-f97fd7426e13"
           (reference "#PWR01") (unit 1)
+        )
+      )
+    )
+  )
+  (symbol (lib_id "Connector:Conn_01x03_Pin") (at 38.735 160.02 0) (unit 1)
+    (in_bom yes) (on_board yes) (dnp no) (fields_autoplaced)
+    (property "Reference" "J1" (at 39.37 152.4 0)
+      (effects (font (size 1.27 1.27)))
+    )
+    (property "Value" "CAM1" (at 39.37 154.94 0)
+      (effects (font (size 1.27 1.27)))
+    )
+    (property "Footprint" "Connector_PinHeader_2.54mm:PinHeader_1x03_P2.54mm_Vertical" (at 38.735 160.02 0)
+      (effects (font (size 1.27 1.27)) hide)
+    )
+    (property "Datasheet" "~" (at 38.735 160.02 0)
+      (effects (font (size 1.27 1.27)) hide)
+    )
+    (pin "3")
+    (pin "1")
+    (pin "2")
+    (instances
+      (project "astrasat1"
+        (path "/9e2da17e-9926-4640-a42c-f97fd7426e13"
+          (reference "J1") (unit 1)
+        )
+      )
+    )
+  )
+  (symbol (lib_id "Connector:Conn_01x03_Pin") (at 38.735 177.8 0) (unit 1)
+    (in_bom yes) (on_board yes) (dnp no) (fields_autoplaced)
+    (property "Reference" "J2" (at 39.37 170.815 0)
+      (effects (font (size 1.27 1.27)))
+    )
+    (property "Value" "CAM2" (at 39.37 173.355 0)
+      (effects (font (size 1.27 1.27)))
+    )
+    (property "Footprint" "Connector_PinHeader_2.54mm:PinHeader_1x03_P2.54mm_Vertical" (at 38.735 177.8 0)
+      (effects (font (size 1.27 1.27)) hide)
+    )
+    (property "Datasheet" "~" (at 38.735 177.8 0)
+      (effects (font (size 1.27 1.27)) hide)
+    )
+    (pin "3")
+    (pin "1")
+    (pin "2")
+    (instances
+      (project "astrasat1"
+        (path "/9e2da17e-9926-4640-a42c-f97fd7426e13"
+          (reference "J2") (unit 1)
         )
       )
@@
         )
       )
+    )
+  )
+  (symbol (lib_id "power:GND1") (at 46.355 162.56 90) (unit 1)
+    (in_bom yes) (on_board yes) (dnp no)
+    (property "Reference" "#PWR023" (at 52.705 162.56 0)
+      (effects (font (size 1.27 1.27)) hide)
+    )
+    (property "Value" "GND1" (at 50.165 162.56 90)
+      (effects (font (size 1.27 1.27)) (justify right))
+    )
+    (property "Footprint" "" (at 46.355 162.56 0)
+      (effects (font (size 1.27 1.27)) hide)
+    )
+    (property "Datasheet" "" (at 46.355 162.56 0)
+      (effects (font (size 1.27 1.27)) hide)
+    )
+    (pin "1")
+    (instances
+      (project "astrasat1"
+        (path "/9e2da17e-9926-4640-a42c-f97fd7426e13"
+          (reference "#PWR023") (unit 1)
+        )
+      )
