File: liberocan1.kicad_pcb (KiCad board)
At the start: 2 copper layers, 118 x 118 mm, 33 parts, among them J1 CAM1, J2 CAM2, SW1 SW_SPDT, U3 DS1302+, U5 Pico, Y1 Crystal

Commit message: update readme
Parts:
- removed the REF** at (151.8, 129.9)
Other:
- board text added: "Licensed with CERN OHL-W v2"
